File: mod-key2.kicad_pcb (KiCad board)
At the start: 2 copper layers, 44 x 30 mm, 13 parts, among them J1 Conn_01x03_Socket

Commit message: Add files via upload
Parts:
- R1, R2, R3, R4, R5, R6: moved to B.Cu
Other:
- board text added: "D"
- board text added: "KEY"
- board text added: "L"
- board text added: "P"
- board text added: "R"
- board text added: "U"
- board text removed: "SW"
